File: kicad/rig/rig.kicad_sch (KiCad schematic)
At the start: 37 parts, among them J1 Baud rate set, J2 TTL-USB, J3 5V DC, SW1 RESET, SW2 POWER, U1 DCJ11, U2 DC319, U3 SN74AHCT14N, U4 74F821SPC, U5 74AHCT541, U6 GAL16V8, Y1 4000 kHz, Y2 614.4 kHz

Commit message: Update KiCad rig for GAL20V8A and late DV capture
Add the GAL20V8A-15LP symbol and complete the matching schematic and routing. Keep separate read and write test points, widen the input power trace to 1.1 mm, and update bypass capacitor placement.

Checked physical pin connectivity, startup bits, current GAL20V8 working-tree logic, and conditional bus timing. PCB DRC and schematic parity pass. Hardware operation remains untested.
Parts:
- removed U6: GAL16V8, Package_DIP:DIP-20_W7.62mm_Socket_LongPads, symbol Logic_Programmable:GAL16V8
- added D2: 1N4148, Diode_THT:D_DO-35_SOD27_P7.62mm_Horizontal, symbol Diode:1N4148
- added R5: 0, Resistor_THT:R_Axial_DIN0207_L6.3mm_D2.5mm_P10.16mm_Horizontal, symbol Device:R
- added TP1: CLK2, Connector_PinHeader_2.54mm:PinHeader_1x01_P2.54mm_Vertical, symbol Connector:TestPoint
- added TP2: ~{INIT}, Connector_PinHeader_2.54mm:PinHeader_1x01_P2.54mm_Vertical, symbol Connector:TestPoint
- added TP3: ~{SCTL}, Connector_PinHeader_2.54mm:PinHeader_1x01_P2.54mm_Vertical, symbol Connector:TestPoint
- added TP4: ~{BUFCTL}, Connector_PinHeader_2.54mm:PinHeader_1x01_P2.54mm_Vertical, symbol Connector:TestPoint
- added TP5: ~{ALE}, Connector_PinHeader_2.54mm:PinHeader_1x01_P2.54mm_Vertical, symbol Connector:TestPoint
- added TP6: LE, Connector_PinHeader_2.54mm:PinHeader_1x01_P2.54mm_Vertical, symbol Connector:TestPoint
- added TP7: DV, Connector_PinHeader_2.54mm:PinHeader_1x01_P2.54mm_Vertical, symbol Connector:TestPoint
- added TP8: ~{OE}, Connector_PinHeader_2.54mm:PinHeader_1x01_P2.54mm_Vertical, symbol Connector:TestPoint
- added TP9: ~{WEL}, Connector_PinHeader_2.54mm:PinHeader_1x01_P2.54mm_Vertical, symbol Connector:TestPoint
- added U6: GAL20V8A-15LP, Package_DIP:DIP-24_W7.62mm_Socket_LongPads, symbol DCJRig:GAL20V8A-15LP
- renumbered R5 to R7, R7 to R8
Connections:
- net A0: now also U6.9 (I8)
- net DV: now also R5.1, TP7.1
- net GND: now also U6.10 (I9), U6.11 (I10), U6.12 (GND), U6.13 (I11/~{OE}), U6.14 (I12), U6.23 (I13); no longer U3.1
- net LAIO0: now also U6.4 (I3)
- net LAIO1: now also U6.3 (I2)
- net LAIO2: now also U6.2 (I1)
- net LAIO3: now also U6.1 (I0/CLK)
- net LBS0: now also U6.5 (I4)
- net LBS1: now also U6.6 (I5)
- net LE: now also TP6.1
- net VCC: now also D2.1 (K), U6.24 (VCC)
- net ~{ALE}: now also TP5.1
- net ~{BUFCTL}: now also TP4.1, U6.8 (I7)
- net ~{GPREAD}: now also U6.22 (I/O7)
- net ~{INIT}: now also TP2.1
- net ~{IO}: now also U6.21 (I/O6)
- net ~{OE}: now also TP8.1, U6.15 (I/O0)
- net ~{SCTL}: now also U3.1, TP3.1, U6.7 (I6)
- net ~{WEL}: now also TP9.1, U6.18 (I/O3)
- net at C8.1, R6.1, R8.2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: now also D2.2 (A)
- net at U3.2: now also R5.2
- net at U1.34 (CLK2): now also TP1.1
- no-connect marks 35 -> 33
Other:
- moved on the sheet: C8, H1, H2, H3, H4, J3, R6, R8, RN1, SW1, SW2, U3A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
